File: eagle/USB-WiFi-Box/usb-wifi-adapter-box.sch (EAGLE design)
At the start: 0 parts

Commit message: inductors and shild ground caps
Parts:
- added C1, C2: (no value), rcl:C-EUC0805
- added CONN1: MINI-USB_SHIELD, dxwifi:MINI-USB_SHIELD
- added L1, L2, L3, L4, L5: (no value), dxwifi:INDUCTOR-BEAD
Connections:
- new net GND: C1.2, C2.2, L1.2
- new net N$1: C2.1, CONN1S.S2
- new net N$2: CONN1G41.4, L2.1
- new net N$3: CONN1G41.3, L3.1
- new net N$4: CONN1G41.2, L4.1
- new net N$5: CONN1G41.1, L5.1
- new net N$6: CONN1G41.5, L1.1
- new net N$7: C1.1, CONN1S.S1
Changed lines of the file:
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@@
 <grid distance="0.1" unitdist="inch" unit="inch" style="lines" multiple="1" display="no" altdistance="0.01" altunitdist="inch" altunit="inch"/>
 <layers>
+<layer number="1" name="Top" color="4" fill="1" visible="no" active="no"/>
+<layer number="16" name="Bottom" color="1" fill="1" visible="no" active="no"/>
+<layer number="17" name="Pads" color="2" fill="1" visible="no" active="no"/>
+<layer number="18" name="Vias" color="2" fill="1" visible="no" active="no"/>
+<layer number="19" name="Unrouted" color="6" fill="1" visible="no" active="no"/>
+<layer number="20" name="Dimension" color="15" fill="1" visible="no" active="no"/>
+<layer number="21" name="tPlace" color="7" fill="1" visible="no" active="no"/>
+<layer number="22" name="bPlace" color="7" fill="1" visible="no" active="no"/>
+<layer number="23" name="tOrigins" color="15" fill="1" visible="no" active="no"/>
+<layer number="24" name="bOrigins" color="15" fill="1" visible="no" active="no"/>
+<layer number="25" name="tNames" color="7" fill="1" visible="no" active="no"/>
+<layer number="26" name="bNames" color="7" fill="1" visible="no" active="no"/>
+<layer number="27" name="tValues" color="7" fill="1" visible="no" active="no"/>
+<layer number="28" name="bValues" color="7" fill="1" visible="no" active="no"/>
+<layer number="29" name="tStop" color="7" fill="3" visible="no" active="no"/>
+<layer number="30" name="bStop" color="7" fill="6" visible="no" active="no"/>
+<layer number="31" name="tCream" color="7" fill="4" visible="no" active="no"/>
+<layer number="32" name="bCream" color="7" fill="5" visible="no" active="no"/>
+<layer number="33" name="tFinish" color="6" fill="3" visible="no" active="no"/>
+<layer number="34" name="bFinish" color="6" fill="6" visible="no" active="no"/>
+<layer number="35" name="tGlue" color="7" fill="4" visible="no" active="no"/>
+<layer number="36" name="bGlue" color="7" fill="5" visible="no" active="no"/>
+<layer number="37" name="tTest" color="7" fill="1" visible="no" active="no"/>
+<layer number="38" name="bTest" color="7" fill="1" visible="no" active="no"/>
+<layer number="39" name="tKeepout" color="4" fill="11" visible="no" active="no"/>
+<layer number="40" name="bKeepout" color="1" fill="11" visible="no" active="no"/>
+<layer number="41" name="tRestrict" color="4" fill="10" visible="no" active="no"/>
+<layer number="42" name="bRestrict" color="1" fill="10" visible="no" active="no"/>
+<layer number="43" name="vRestrict" color="2" fill="10" visible="no" active="no"/>
+<layer number="44" name="Drills" color="7" fill="1" visible="no" active="no"/>
+<layer number="45" name="Holes" color="7" fill="1" visible="no" active="no"/>
+<layer number="46" name="Milling" color="3" fill="1" visible="no" active="no"/>
+<layer number="47" name="Measures" color="7" fill="1" visible="no" active="no"/>
+<layer number="48" name="Document" color="7" fill="1" visible="no" active="no"/>
+<layer number="49" name="Reference" color="7" fill="1" visible="no" active="no"/>
+<layer number="51" name="tDocu" color="7" fill="1" visible="no" active="no"/>
+<layer number="52" name="bDocu" color="7" fill="1" visible="no" active="no"/>
 <layer number="91" name="Nets" color="2" fill="1" visible="yes" active="yes"/>
 <layer number="92" name="Busses" color="1" fill="1" visible="yes" active="yes"/>
@@
 </classes>
 <parts>
+<part name="CONN1" library="dxwifi" deviceset="MINI-USB_SHIELD" device=""/>
+<part name="L1" library="dxwifi" deviceset="INDUCTOR-BEAD" device=""/>
+<part name="L2" library="dxwifi" deviceset="INDUCTOR-BEAD" device=""/>
+<part name="L3" library="dxwifi" deviceset="INDUCTOR-BEAD" device=""/>
+<part name="L4" library="dxwifi" deviceset="INDUCTOR-BEAD" device=""/>
+<part name="L5" library="dxwifi" deviceset="INDUCTOR-BEAD" device=""/>
+<part name="C1" library="rcl" deviceset="C-EU" device="C0805"/>
+<part name="C2" library="rcl" deviceset="C-EU" device="C0805"/>
+<part name="SUPPLY1" library="supply2" deviceset="GND" device=""/>
 </parts>
 <sheets>
@@
 </plain>
 <instances>
+<instance part="CONN1" gate="G41" x="10.16" y="38.1" smashed="yes" rot="MR0">
+<attribute name="VALUE" x="0" y="30.48" size="1.778" layer="96" font="vector" rot="MR90"/>
+</instance>
+<instance part="L1" gate="G$1" x="20.32" y="17.78" rot="R270"/>
+<instance part="L2" gate="G$1" x="30.48" y="35.56"/>
+<instance part="L3" gate="G$1" x="25.4" y="38.1"/>
+<instance part="L4" gate="G$1" x="30.48" y="40.64"/>
+<instance part="L5" gate="G$1" x="22.86" y="43.18"/>
+<instance part="C1" gate="G$1" x="7.62" y="20.32"/>
+<instance part="C2" gate="G$1" x="12.7" y="20.32"/>
+<instance part="SUPPLY1" gate="GND" x="17.78" y="12.7"/>
+<instance part="CONN1" gate="S" x="12.7" y="27.94"/>
 </instances>
 <busses>
 </busses>
 <nets>
+<net name="N$2" class="0">
+<segment>
+<pinref part="L2" gate="G$1" pin="1"/>
+<pinref part="CONN1" gate="G41" pin="4"/>
+<wire x1="15.24" y1="35.56" x2="25.4" y2="35.56" width="0.1524" layer="91"/>
+</segment>
+</net>
+<net name="N$3" class="0">
+<segment>
+<pinref part="CONN1" gate="G41" pin="3"/>
+<pinref part="L3" gate="G$1" pin="1"/>
+<wire x1="15.24" y1="38.1" x2="20.32" y2="38.1" width="0.1524" layer="91"/>
+</segment>
+</net>
+<net name="N$4" class="0">
+<segment>
+<pinref part="CONN1" gate="G41" pin="2"/>
+<pinref part="L4" gate="G$1" pin="1"/>
+<wire x1="15.24" y1="40.64" x2="25.4" y2="40.64" width="0.1524" layer="91"/>
+</segment>
+</net>
+<net name="N$5" class="0">
+<segment>
+<pinref part="CONN1" gate="G41" pin="1"/>
+<pinref part="L5" gate="G$1" pin="1"/>
+<wire x1="15.24" y1="43.18" x2="17.78" y2="43.18" width="0.1524" layer="91"/>
+</segment>
+</net>
+<net name="GND" class="0">
+<segment>
+<pinref part="C1" gate="G$1" pin="2"/>
+<pinref part="C2" gate="G$1" pin="2"/>
+<wire x1="7.62" y1="15.24" x2="12.7" y2="15.24" width="0.1524" layer="91"/>
+<pinref part="L1" gate="G$1" pin="2"/>
+<wire x1="12.7" y1="15.24" x2="20.32" y2="15.24" width="0.1524" layer="91"/>
+<junction x="12.7" y="15.24"/>
+<pinref part="SUPPLY1" gate="GND" pin="GND"/>
+<junction x="20.32" y="15.24"/>
+<wire x1="20.32" y1="15.24" x2="17.78" y2="15.24" width="0.1524" layer="91"/>
+</segment>
+</net>
+<net name="N$6" class="0">
+<segment>
+<pinref part="CONN1" gate="G41" pin="5"/>
+<pinref part="L1" gate="G$1" pin="1"/>
+<wire x1="15.24" y1="33.02" x2="20.32" y2="33.02" width="0.1524" layer="91"/>
+<wire x1="20.32" y1="33.02" x2="20.32" y2="22.86" width="0.1524" layer="91"/>
+</segment>
+</net>
+<net name="N$1" class="0">
+<segment>
+<pinref part="CONN1" gate="S" pin="S2"/>
+<pinref part="C2" gate="G$1" pin="1"/>
+<wire x1="12.7" y1="25.4" x2="12.7" y2="22.86" width="0.1524" layer="91"/>
+</segment>
+</net>
+<net name="N$7" class="0">
+<segment>
+<pinref part="CONN1" gate="S" pin="S1"/>
+<wire x1="10.16" y1="25.4" x2="7.62" y2="25.4" width="0.1524" layer="91"/>
+<pinref part="C1" gate="G$1" pin="1"/>
+<wire x1="7.62" y1="25.4" x2="7.62" y2="22.86" width="0.1524" layer="91"/>
+</segment>
+</net>
 </nets>
 </sheet>
